Commit message: changed cam plugin

File: arucobot_description/urdf/gazebo_control.xacro (robot description, xacro)
@@ -21,3 +21,51 @@
       </plugin>
    </gazebo>
+   <!-- CAMERA -->
+<gazebo reference="mr_robot/base_link/depth_camera1">
+  <sensor name="camera" type="camera">
+        <camera>
+          <horizontal_fov>1.51844</horizontal_fov>
+          <image>
+            <width>640</width>
+            <height>480</height>
+            <format>RGB_INT8</format>
+          </image>
+          <clip>
+            <near>0.1</near>
+            <far>100</far>
+          </clip>
+          <noise>
+            <type>gaussian</type>
+            <mean>0.0</mean>
+            <stddev>0.007</stddev>
+          </noise>
+        </camera>
+        <always_on>1</always_on>
+        <update_rate>30</update_rate>
+        <visualize>1</visualize>
+        <topic>camera</topic>
+      </sensor>
+</gazebo>
+<!-- Depth camera -->
+<gazebo reference="mr_robot/base_link/depth_camera1">
+  <sensor name="depth_camera1" type="depth_camera">
+        <always_on>1</always_on>
+        <enable_metrics>1</enable_metrics>
+        <topic>depth_camera</topic>
+        <update_rate>10</update_rate>
+        <visualize>1</visualize>
+        <camera>
+          <horizontal_fov>1.05</horizontal_fov>
+          <image>
+            <width>640</width>
+            <height>480</height>
+            <format>R_FLOAT32</format>
+          </image>
+          <clip>
+            <near>0.1</near>
+            <far>10.0</far>
+          </clip>
+        </camera>
+      </sensor>
+</gazebo>
 </robot>

File: arucobot_description/urdf/robot.urdf.xacro (robot description, xacro)
@@ -3,3 +3,4 @@
     <xacro:include filename="robot_core.xacro" />
     <xacro:include filename="gazebo_control.xacro" />
+    <xacro:include filename="materials.xacro" />
 </robot>

File: arucobot_description/urdf/robot_core.xacro (robot description, xacro)
@@ -2,16 +2,4 @@
 <robot xmlns:xacro="http://www.ros.org/wiki/xacro" >
     <xacro:include filename="inertial_macros.xacro"/>
-    <material name="white">
-        <color rgba="1 1 1 1" />
-    </material>
-    <material name="orange">
-        <color rgba="1 0.3 0.1 1"/>
-    </material>
-    <material name="blue">
-        <color rgba="0.2 0.2 1 1"/>
-    </material>
-    <material name="black">
-        <color rgba="0 0 0 1"/>
-    </material>
     <!-- BASE LINK -->
     <link name="base_link">
@@ -109,61 +97,31 @@
         </xacro:inertial_sphere>
     </link>
-<joint name="camera_joint" type="fixed">
-    <axis xyz="0 0 0"/>
-    <origin rpy="0 0 0" xyz="0.27 0 0.14"/>
-    <parent link="base_link"/>
-    <child link="camera_link"/>
-  </joint>
-<joint name="camera_optical_joint" type="fixed">
-    <parent link="camera_link"/>
-    <child link="camera_link_optical"/>
-    <origin xyz="0 0 0" rpy="${-pi/2} 0 ${-pi/2}"/>
-  </joint>
-<link name="camera_link_optical"></link>
- <link name="camera_link">
-    <collision>
-      <origin rpy="0 0 0" xyz="0 0 0"/>
-      <geometry>
-        <box size="0.05 0.05 0.05"/>
-      </geometry>
-    </collision>
-    <visual>
-      <origin rpy="0 0 0" xyz="0 0 0"/>     <!-- roll pitch and yaw in radians and xyz in meters-->
-      <geometry>
-        <box size="0.05 0.05 0.05"/>
-      </geometry>
-      <material name="red"/>
-    </visual>
-    <inertial>
-      <mass value="1e-5"/>
-      <origin rpy="0 0 0" xyz="0 0 0"/>
-      <inertia ixx="1e-6" ixy="0" ixz="0" iyy="1e-6" iyz="0" izz="1e-6"/>
-    </inertial>
-  </link>
-  <joint name="depth_camera_joint" type="fixed">
-    <axis xyz="0 0 0" />
-    <origin xyz="0.27 0.1 0.14" rpy="0 0 0"/>
-    <parent link="base_link"/>
-    <child link="mr_robot/base_link/depth_camera"/>
-  </joint>
-  <link name="mr_robot/base_link/depth_camera">
-    <collision>
-      <origin xyz="0 0 0" rpy="0 0 0"/>
-      <geometry>
-    <box size="0.05 0.05 0.05"/>
-      </geometry>
-    </collision>
-    <visual>
-      <origin xyz="0 0 0" rpy="0 0 0"/>
-      <geometry>
-    <box size="0.05 0.05 0.05"/>
-      </geometry>
-      <material name="dark_blue"/>
-    </visual>
-    <inertial>
-      <mass value="1e-5" />
-      <origin xyz="0 0 0" rpy="0 0 0"/>
-      <inertia ixx="1e-6" ixy="0" ixz="0" iyy="1e-6" iyz="0" izz="1e-6" />
-    </inertial>
-  </link>
+    <xacro:property name="camera_link" value="0.05" /> <!-- Size of square 'camera' box -->
+    <joint name="camera_joint" type="fixed">
+        <axis xyz="0 1 0" />
+        <origin xyz="0.2 0.0 0.17" rpy="0 0 0"/>
+        <parent link="base_link"/>
+        <child link="mr_robot/base_link/depth_camera1"/>
+    </joint>
+    <!-- Camera -->
+    <link name="mr_robot/base_link/depth_camera1">
+        <collision>
+        <origin xyz="0 0 0" rpy="0 0 0"/>
+        <geometry>
+        <box size="${camera_link} ${camera_link} ${camera_link}"/>
+        </geometry>
+        </collision>
+        <visual>
+        <origin xyz="0 0 0" rpy="0 0 0"/>
+        <geometry>
+        <box size="${camera_link} ${camera_link} ${camera_link}"/>
+        </geometry>
+        <material name="red"/>
+        </visual>
+        <inertial>
+        <mass value="1e-5" />
+        <origin xyz="0 0 0" rpy="0 0 0"/>
+        <inertia ixx="1e-6" ixy="0" ixz="0" iyy="1e-6" iyz="0" izz="1e-6" />
+        </inertial>
+    </link>
 </robot>

Commit message: camera working

File: arucobot_description/urdf/gazebo_control.xacro (robot description, xacro)
@@ -22,39 +22,37 @@
    </gazebo>
    <!-- CAMERA -->
-<gazebo reference="mr_robot/base_link/depth_camera1">
-  <sensor name="camera" type="camera">
-        <camera>
-          <horizontal_fov>1.51844</horizontal_fov>
-          <image>
-            <width>640</width>
-            <height>480</height>
-            <format>RGB_INT8</format>
-          </image>
-          <clip>
-            <near>0.1</near>
-            <far>100</far>
-          </clip>
-          <noise>
-            <type>gaussian</type>
-            <mean>0.0</mean>
-            <stddev>0.007</stddev>
-          </noise>
-        </camera>
-        <always_on>1</always_on>
-        <update_rate>30</update_rate>
-        <visualize>1</visualize>
-        <topic>camera</topic>
-      </sensor>
-</gazebo>
-<!-- Depth camera -->
-<gazebo reference="mr_robot/base_link/depth_camera1">
-  <sensor name="depth_camera1" type="depth_camera">
-        <always_on>1</always_on>
-        <enable_metrics>1</enable_metrics>
-        <topic>depth_camera</topic>
+<gazebo reference="arucobot/base_link/depth_camera1">
+<plugin filename="gz-harmonic-camera-system" name="gz::harmonic::systems::CameraSystem"/>
+    <sensor type="camera" name="camera">
+      <visualize>true</visualize>
+      <always_on>true</always_on>
+      <update_rate>10.0</update_rate>
+      <camera name="head">
+        <!-- <camera_info_topic>camera/camera_info</camera_info_topic> -->
+        <horizontal_fov>1.3962634</horizontal_fov>  <!-- 80 degrees-->
+        <image>
+          <width>800</width>
+          <height>800</height>
+          <format>R8G8B8</format>   <!-- RGB WITH 8 BITS PER CHANNEL-->
+        </image>
+        <clip>
+          <near>0.02</near>
+          <far>300</far>
+        </clip>
+      </camera>
+      <topic>camera/image_raw</topic>
+      <gz_frame_id>camera_link_optical</gz_frame_id>
+    </sensor>
+  </gazebo>
+<gazebo reference="arucobot/base_link/depth_camera1">
+<plugin filename="gz-sim-depth-camera-system" name="gz::sim::systems::DepthCamera"/>
+  <sensor type="depth_camera" name="depth_camera">
+        <visualize>true</visualize>
+        <always_on>true</always_on>
+        <enable_metrics>true</enable_metrics>
         <update_rate>10</update_rate>
-        <visualize>1</visualize>
-        <camera>
-          <horizontal_fov>1.05</horizontal_fov>
+        <camera name = "Deep">
+          <camera_info_topic>depth_camera/depth_camera_info</camera_info_topic>
+          <horizontal_fov>1.3962634</horizontal_fov>
           <image>
             <width>640</width>
@@ -63,8 +61,10 @@
           </image>
           <clip>
-            <near>0.1</near>
-            <far>10.0</far>
+            <near>0.02</near>
+            <far>300</far>
           </clip>
         </camera>
+        <topic>depth_camera</topic>
+        <gz_frame_id>camera_link_optical</gz_frame_id>
       </sensor>
 </gazebo>

File: arucobot_description/urdf/robot_core.xacro (robot description, xacro)
@@ -102,8 +102,8 @@
         <origin xyz="0.2 0.0 0.17" rpy="0 0 0"/>
         <parent link="base_link"/>
-        <child link="mr_robot/base_link/depth_camera1"/>
+        <child link="arucobot/base_link/depth_camera1"/>
     </joint>
     <!-- Camera -->
-    <link name="mr_robot/base_link/depth_camera1">
+    <link name="arucobot/base_link/depth_camera1">
         <collision>
         <origin xyz="0 0 0" rpy="0 0 0"/>

Commit message: added lidar

File: arucobot_description/urdf/gazebo_control.xacro (robot description, xacro)
@@ -67,3 +67,34 @@
       </sensor>
 </gazebo>
+<gazebo reference="arucobot/base_link/gpu_lidar">
+  <sensor name='gpu_lidar' type='gpu_lidar'>"
+    <pose relative_to='arucobot/base_link/gpu_lidar'>0.001 0.006 0.1155 0 0 0</pose>
+    <frame_id>arucobot/base_link/gpu_lidar</frame_id>
+    <topic>/laser/scan</topic>
+    <update_rate>10</update_rate>
+    <ray>
+        <scan>
+            <horizontal>
+                <samples>300</samples>
+                <resolution>1</resolution>
+                <min_angle>-3.14</min_angle>
+                <max_angle>3.14</max_angle>
+            </horizontal>
+            <vertical>
+                <samples>1</samples>
+                <resolution>0.01</resolution>
+                <min_angle>0</min_angle>
+                <max_angle>0</max_angle>
+            </vertical>
+        </scan>
+        <range>
+            <min>0.01</min>
+            <max>10.0</max>
+            <resolution>0.01</resolution>
+        </range>
+    </ray>
+    <always_on>1</always_on>
+    <visualize>true</visualize>
+</sensor>
+</gazebo>
 </robot>

File: arucobot_description/urdf/robot_core.xacro (robot description, xacro)
@@ -100,5 +100,5 @@
     <joint name="camera_joint" type="fixed">
         <axis xyz="0 1 0" />
-        <origin xyz="0.2 0.0 0.17" rpy="0 0 0"/>
+        <origin xyz="0.2 0.0 0.1" rpy="0 0 0"/>
         <parent link="base_link"/>
         <child link="arucobot/base_link/depth_camera1"/>
@@ -125,3 +125,27 @@
         </inertial>
     </link>
+ <!-- LIDAR SENSOR -->
+    <joint name="lidar_joint" type="fixed">
+        <parent link="base_link"/>
+        <child link="arucobot/base_link/gpu_lidar"/>
+        <origin xyz="0.04 0 0.18" rpy="0 0 0"/>
+    </joint>
+    <link name="arucobot/base_link/gpu_lidar">
+        <visual>
+            <geometry>
+                <cylinder radius="0.03" length="0.06"/>
+            </geometry>
+            <material name="black"/>
+        </visual>
+        <collision>
+            <geometry>
+                <cylinder radius="0.03" length="0.06"/>
+            </geometry>
+        </collision>
+        <inertial>
+            <mass value="0.05"/>
+            <origin xyz="0 0 0" rpy="0 0 0"/>
+            <inertia ixx="1e-6" ixy="0" ixz="0" iyy="1e-6" iyz="0" izz="1e-6"/>
+        </inertial>
+    </link>
 </robot>

Commit message: mapping done

File: arucobot_description/urdf/gazebo_control.xacro (robot description, xacro)
@@ -1,5 +1,5 @@
 <?xml version="1.0"?>
 <robot xmlns:xacro="http://www.ros.org/wiki/xacro">
-   <gazebo>
+   <!-- <gazebo>
       <plugin filename="gz-sim-diff-drive-system" name="gz::sim::systems::DiffDrive">
          <right_joint>right_wheel_joint</right_joint>
@@ -7,28 +7,43 @@
          <wheel_separation>0.35</wheel_separation>
          <wheel_diameter>0.1</wheel_diameter>
-         <max_linear_acceleration>10</max_linear_acceleration>
+         <max_linear_acceleration>3</max_linear_acceleration>
          <topic>cmd_vel</topic>
-         <odom_topic>odom</odom_topic>
-         <frame_id>odom</frame_id>
          <child_frame_id>base_link</child_frame_id>
          <odom_publisher_frequency>100</odom_publisher_frequency>
          <tf_topic>/tf</tf_topic>
+         <publish_odom>true</publish_odom>
+         <publish_odom_tf>false</publish_odom_tf>
+         <publish_wheel_tf>true</publish_wheel_tf>
+         <odometry_frame>odom</odometry_frame>
+         <robot_base_frame>base_link</robot_base_frame>
       </plugin>
       <plugin filename="gz-sim-joint-state-publisher-system" name="gz::sim::systems::JointStatePublisher">
-         <topic>joint_states</topic>
+         <topic>/joint_states</topic>
          <joint_name>right_wheel_joint</joint_name>
          <joint_name>left_wheel_joint</joint_name>
       </plugin>
-   </gazebo>
-   <gazebo>
+   </gazebo> -->
+	<gazebo>
+		<plugin filename="gz-sim-diff-drive-system"
+			name="gz::sim::systems::DiffDrive">
+			<left_joint>left_wheel_joint</left_joint>
+    		<right_joint>right_wheel_joint</right_joint>
+    		<wheel_separation>0.45</wheel_separation>
+    		<wheel_radius>0.06</wheel_radius>
+			<topic>cmd_vel_gz</topic>
+			<odom_topic>odom_gz</odom_topic>
+			<tf_topic>tf_gz</tf_topic>
+    	</plugin>
+	</gazebo>
+	<gazebo>
       <plugin
         filename="gz-sim-odometry-publisher-system"
         name="gz::sim::systems::OdometryPublisher">
-        <odom_frame>odom</odom_frame>
-        <robot_base_frame>base_link</robot_base_frame>
-        <odom_topic>/odom</odom_topic>
-        <tf_topic>/tf</tf_topic>
+		<odom_frame>odom</odom_frame>
+		<robot_base_frame>base_link</robot_base_frame>
+		<odom_topic>/odom</odom_topic>
+		<tf_topic>/tf</tf_topic>
       </plugin>
-    </gazebo>
+	</gazebo>
    <!-- CAMERA -->
 <gazebo reference="arucobot/base_link/depth_camera1">

File: arucobot_description/urdf/robot_core.xacro (robot description, xacro)
@@ -4,4 +4,16 @@
     <!-- BASE LINK -->
     <link name="base_link">
+          <inertial>
+    <origin xyz="0.00024062344110785007 -0.00531572402780089 -0.10823524150435863" rpy="0 0 0"/>
+    <mass value="19.729806517747196"/>
+    <inertia ixx="0.871968" iyy="0.872497" izz="1.726537" ixy="0.000808" iyz="0.001686" ixz="0.000142"/>
+  </inertial>
+  <visual>
+    <origin xyz="0 0 0" rpy="0 0 0"/>
+    <material name="silver"/>
+  </visual>
+  <collision>
+    <origin xyz="0 0 0" rpy="0 0 0"/>
+  </collision>
     </link>
     <!-- CHASSIS LINK -->
@@ -25,5 +37,5 @@
             </geometry>
         </collision>
-        <xacro:inertial_box mass="0.5" x="0.3" y="0.3" z="0.15">
+        <xacro:inertial_box mass="2.0" x="0.3" y="0.3" z="0.15">
             <origin xyz="0.15 0 0.075" rpy="0 0 0"/>
         </xacro:inertial_box>
@@ -93,6 +105,6 @@
             </geometry>
         </collision>
-        <xacro:inertial_sphere mass="0.1" radius="0.05">
-            <origin xyz="0 0 0" rpy="0 0 0"/>
+        <xacro:inertial_sphere mass="0.5" radius="0.05">
+            <origin xyz="0.24 0 0" rpy="0 0 0"/>
         </xacro:inertial_sphere>
     </link>
