Commit message: fixed nav orientation, odom rough

File: vanir_description/urdf/robot_core.xacro (robot description, xacro)
@@ -9,5 +9,5 @@
     <!-- Part base_link -->
     <visual>
-      <origin xyz="0.0684338 0.00840189 0.000920176" rpy="0 -0 1.5708"/>
+      <origin xyz="0.0684338 0.00840189 0.000920176" rpy="0 -0 -1.5708"/>
       <geometry>
         <mesh filename="file://$(find vanir_description)/meshes/base_link.stl"/>

Commit message: repositioned bot and tuned

File: vanir_description/urdf/robot_core.xacro (robot description, xacro)
@@ -9,5 +9,5 @@
     <!-- Part base_link -->
     <visual>
-      <origin xyz="0.0684338 0.00840189 0.000920176" rpy="0 -0 -1.5708"/>
+      <origin xyz="0.0684338 0.00840189 0.000920176" rpy="0 -0 1.5708"/>
       <geometry>
         <mesh filename="file://$(find vanir_description)/meshes/base_link.stl"/>
