Commit message: renamed bot

File: vanir_description/urdf/gazebo_control.xacro (robot description, xacro)
@@ -45,5 +45,5 @@
 	</gazebo>
    <!-- CAMERA -->
-<gazebo reference="arucobot/base_link/depth_camera1">
+<gazebo reference="vanir/base_link/depth_camera1">
 <plugin filename="gz-harmonic-camera-system" name="gz::harmonic::systems::CameraSystem"/>
     <sensor type="camera" name="camera">
@@ -69,5 +69,5 @@
   </gazebo>
 <!-- Depth camera -->
-<gazebo reference="arucobot/base_link/depth_camera1">
+<gazebo reference="vanir/base_link/depth_camera1">
   <sensor name="depth_camera1" type="depth_camera">
         <always_on>1</always_on>
@@ -90,8 +90,8 @@
       </sensor>
 </gazebo>
-<gazebo reference="arucobot/base_link/gpu_lidar">
+<gazebo reference="vanir/base_link/gpu_lidar">
   <sensor name='gpu_lidar' type='gpu_lidar'>"
-    <pose relative_to='arucobot/base_link/gpu_lidar'>0.001 0.006 0.1155 0 0 0</pose>
-    <frame_id>arucobot/base_link/gpu_lidar</frame_id>
+    <pose relative_to='vanir/base_link/gpu_lidar'>0.001 0.006 0.1155 0 0 0</pose>
+    <frame_id>vanir/base_link/gpu_lidar</frame_id>
     <topic>/laser/scan</topic>
     <update_rate>10</update_rate>

File: vanir_description/urdf/robot_core.xacro (robot description, xacro)
@@ -114,8 +114,8 @@
         <origin xyz="0.2 0.0 0.1" rpy="0 0 0"/>
         <parent link="base_link"/>
-        <child link="arucobot/base_link/depth_camera1"/>
+        <child link="vanir/base_link/depth_camera1"/>
     </joint>
     <!-- Camera -->
-    <link name="arucobot/base_link/depth_camera1">
+    <link name="vanir/base_link/depth_camera1">
         <collision>
         <origin xyz="0 0 0" rpy="0 0 0"/>
@@ -140,8 +140,8 @@
     <joint name="lidar_joint" type="fixed">
         <parent link="base_link"/>
-        <child link="arucobot/base_link/gpu_lidar"/>
+        <child link="vanir/base_link/gpu_lidar"/>
         <origin xyz="0.04 0 0.18" rpy="0 0 0"/>
     </joint>
-    <link name="arucobot/base_link/gpu_lidar">
+    <link name="vanir/base_link/gpu_lidar">
         <visual>
             <geometry>

Commit message: fixed wheel origin

File: vanir_description/urdf/gazebo_control.xacro (robot description, xacro)
@@ -27,6 +27,6 @@
 		<plugin filename="gz-sim-diff-drive-system"
 			name="gz::sim::systems::DiffDrive">
-			<left_joint>left_wheel_joint</left_joint>
-    		<right_joint>right_wheel_joint</right_joint>
+			<left_joint>wheel_l</left_joint>
+    		<right_joint>wheel_r</right_joint>
     		<wheel_separation>0.45</wheel_separation>
     		<wheel_radius>0.06</wheel_radius>

File: vanir_description/urdf/robot.urdf.xacro (robot description, xacro)
@@ -3,4 +3,3 @@
     <xacro:include filename="robot_core.xacro" />
     <xacro:include filename="gazebo_control.xacro" />
-    <xacro:include filename="materials.xacro" />
 </robot>

File: vanir_description/urdf/robot_core.xacro (robot description, xacro)
@@ -1,163 +1,164 @@
 <?xml version="1.0"?>
 <robot xmlns:xacro="http://www.ros.org/wiki/xacro" >
-    <xacro:include filename="inertial_macros.xacro"/>
-    <!-- BASE LINK -->
-    <link name="base_link">
-          <inertial>
-    <origin xyz="0.00024062344110785007 -0.00531572402780089 -0.10823524150435863" rpy="0 0 0"/>
-    <mass value="19.729806517747196"/>
-    <inertia ixx="0.871968" iyy="0.872497" izz="1.726537" ixy="0.000808" iyz="0.001686" ixz="0.000142"/>
-  </inertial>
+  <link name="base_link">
+    <inertial>
+      <origin xyz="0.000219763 -0.000623028 0.0710795" rpy="0 0 0"/>
+      <mass value="92.4179"/>
+      <inertia ixx="3.16969" ixy="2.70317e-05" ixz="1.26673e-06" iyy="1.30381" iyz="0.00479148" izz="3.85167"/>
+    </inertial>
+    <!-- Part front_caster -->
+    <visual>
+      <origin xyz="0.000218796 0.00283755 0.000920176" rpy="0 -0 0"/>
+      <geometry>
+        <mesh filename="file://$(find vanir_description)/meshes/front_caster.stl"/>
+      </geometry>
+      <material name="front_caster_material">
+        <color rgba="0.301961 0.301961 0.301961 1.0"/>
+      </material>
+    </visual>
+    <collision>
+      <origin xyz="0.000218796 0.00283755 0.000920176" rpy="0 -0 0"/>
+      <geometry>
+        <mesh filename="file://$(find vanir_description)/meshes/front_caster.stl"/>
+      </geometry>
+    </collision>
+    <!-- Part rear_caster -->
+    <visual>
+      <origin xyz="0.000218796 0.00276511 0.000920176" rpy="0 -0 0"/>
+      <geometry>
+        <mesh filename="file://$(find vanir_description)/meshes/rear_caster.stl"/>
+      </geometry>
+      <material name="rear_caster_material">
+        <color rgba="0.301961 0.301961 0.301961 1.0"/>
+      </material>
+    </visual>
+    <collision>
+      <origin xyz="0.000218796 0.00276511 0.000920176" rpy="0 -0 0"/>
+      <geometry>
+        <mesh filename="file://$(find vanir_description)/meshes/rear_caster.stl"/>
+      </geometry>
+    </collision>
+    <!-- Part base_link -->
+    <visual>
+      <origin xyz="0.000218796 4.86233e-05 0.000920176" rpy="0 -0 0"/>
+      <geometry>
+        <mesh filename="file://$(find vanir_description)/meshes/base_link.stl"/>
+      </geometry>
+      <material name="base_link_material">
+        <color rgba="0.917647 0.917647 0.917647 1.0"/>
+      </material>
+    </visual>
+    <collision>
+      <origin xyz="0.000218796 4.86233e-05 0.000920176" rpy="0 -0 0"/>
+      <geometry>
+        <mesh filename="file://$(find vanir_description)/meshes/base_link.stl"/>
+      </geometry>
+    </collision>
+  </link>
+  <!-- Link dof_wheel_r -->
+  <link name="dof_wheel_r">
+    <inertial>
+      <origin xyz="3.28288e-18 -8.8737e-19 -0.025" rpy="0 0 0"/>
+      <mass value="0.908215"/>
+      <inertia ixx="0.00138266" ixy="0" ixz="0" iyy="0.00138266" iyz="0" izz="0.0023869"/>
+    </inertial>
+    <visual>
+      <origin xyz="0 -4.44523e-18 0.1625" rpy="-1.5708 -1.5708 0"/>
+      <geometry>
+        <mesh filename="file://$(find vanir_description)/meshes/dof_wheel_r.stl"/>
+      </geometry>
+      <material name="dof_wheel_r_material">
+        <color rgba="0.301961 0.301961 0.301961 1.0"/>
+      </material>
+    </visual>
+    <collision>
+      <origin xyz="0 -4.44523e-18 0.1625" rpy="-1.5708 -1.5708 0"/>
+      <geometry>
+        <mesh filename="file://$(find vanir_description)/meshes/dof_wheel_r.stl"/>
+      </geometry>
+    </collision>
+  </link>
+  <joint name="wheel_r" type="continuous">
+    <origin xyz="-0.162281 4.86233e-05 -0.005" rpy="1.5708 -0 1.5708"/>
+    <parent link="base_link"/>
+    <child link="dof_wheel_r"/>
+    <axis xyz="0 0 1"/>
+    <limit effort="10" velocity="10"/>
+  </joint>
+  <!-- Link dof_wheel_l -->
+  <link name="dof_wheel_l">
+    <inertial>
+      <origin xyz="-3.28288e-18 -1.9388e-18 -0.025" rpy="0 0 0"/>
+      <mass value="0.908215"/>
+      <inertia ixx="0.00138266" ixy="0" ixz="0" iyy="0.00138266" iyz="0" izz="0.0023869"/>
+    </inertial>
+    <visual>
+      <origin xyz="1.38778e-17 4.44523e-18 0.1625" rpy="1.5708 1.5708 0"/>
+      <geometry>
+        <mesh filename="file://$(find vanir_description)/meshes/dof_wheel_l.stl"/>
+      </geometry>
+      <material name="dof_wheel_l_material">
+        <color rgba="0.301961 0.301961 0.301961 1.0"/>
+      </material>
+    </visual>
+    <collision>
+      <origin xyz="1.38778e-17 4.44523e-18 0.1625" rpy="1.5708 1.5708 0"/>
+      <geometry>
+        <mesh filename="file://$(find vanir_description)/meshes/dof_wheel_l.stl"/>
+      </geometry>
+    </collision>
+  </link>
+  <joint name="wheel_l" type="continuous">
+    <origin xyz="0.162719 4.86233e-05 -0.005" rpy="-1.5708 -0 1.5708"/>
+    <parent link="base_link"/>
+    <child link="dof_wheel_l"/>
+    <axis xyz="0 0 -1"/>
+    <limit effort="10" velocity="10"/>
+  </joint>
+  <!-- CAMERA LINK -->
+<link name="vanir/base_link/depth_camera1">
   <visual>
     <origin xyz="0 0 0" rpy="0 0 0"/>
-    <material name="silver"/>
+    <geometry>
+      <mesh filename="file://$(find vanir_description)/meshes/camera.stl"/>
+    </geometry>
+    <material name="camera_material">
+      <color rgba="0.301961 0.290196 0.262745 1.0"/>
+    </material>
   </visual>
   <collision>
     <origin xyz="0 0 0" rpy="0 0 0"/>
+    <geometry>
+      <mesh filename="file://$(find vanir_description)/meshes/camera.stl"/>
+    </geometry>
   </collision>
-    </link>
-    <!-- CHASSIS LINK -->
-    <joint name="chassis_joint" type="fixed">
-        <parent link="base_link"/>
-        <child link="chassis"/>
-        <origin xyz="-0.1 0 0"/>
-    </joint>
-    <link name="chassis">
-        <visual>
-            <origin xyz="0.15 0 0.075"/>
-            <geometry>
-                <box size="0.3 0.3 0.15"/>
-            </geometry>
-            <material name="white"/>
-        </visual>
-        <collision>
-            <origin xyz="0.15 0 0.075"/>
-            <geometry>
-                <box size="0.3 0.3 0.15"/>
-            </geometry>
-        </collision>
-        <xacro:inertial_box mass="2.0" x="0.3" y="0.3" z="0.15">
-            <origin xyz="0.15 0 0.075" rpy="0 0 0"/>
-        </xacro:inertial_box>
-    </link>
-    <!-- LEFT WHEEL LINK -->
-    <joint name="left_wheel_joint" type="continuous">
-        <parent link="base_link"/>
-        <child link="left_wheel"/>
-        <origin xyz="0 0.175 0" rpy="-${pi/2} 0 0" />
-        <axis xyz="0 0 1"/>
-    </joint>
-    <link name="left_wheel">
-        <visual>
-            <geometry>
-                <cylinder radius="0.05" length="0.04"/>
-            </geometry>
-            <material name="blue"/>
-        </visual>
-        <collision>
-            <geometry>
-                <cylinder radius="0.05" length="0.04"/>
-            </geometry>
-        </collision>
-        <xacro:inertial_cylinder mass="0.1" length="0.04" radius="0.05">
-            <origin xyz="0 0 0" rpy="0 0 0"/>
-        </xacro:inertial_cylinder>
-    </link>
-    <!-- RIGHT WHEEL LINK -->
-    <joint name="right_wheel_joint" type="continuous">
-        <parent link="base_link"/>
-        <child link="right_wheel"/>
-        <origin xyz="0 -0.175 0" rpy="${pi/2} 0 0" />
-        <axis xyz="0 0 -1"/>
-    </joint>
-    <link name="right_wheel">
-        <visual>
-            <geometry>
-                <cylinder radius="0.05" length="0.04"/>
-            </geometry>
-            <material name="blue"/>
-        </visual>
-        <collision>
-            <geometry>
-                <cylinder radius="0.05" length="0.04"/>
-            </geometry>
-        </collision>
-        <xacro:inertial_cylinder mass="0.1" length="0.04" radius="0.05">
-            <origin xyz="0 0 0" rpy="0 0 0"/>
-        </xacro:inertial_cylinder>
-    </link>
-    <!-- CASTER WHEEL LINK -->
-    <joint name="caster_wheel_joint" type="fixed">
-        <parent link="chassis"/>
-        <child link="caster_wheel"/>
-        <origin xyz="0.24 0 0"/>
-    </joint>
-    <link name="caster_wheel">
-        <visual>
-            <geometry>
-                <sphere radius="0.05"/>
-            </geometry>
-            <material name="black"/>
-        </visual>
-        <collision>
-            <geometry>
-                <sphere radius="0.05"/>
-            </geometry>
-        </collision>
-        <xacro:inertial_sphere mass="0.5" radius="0.05">
-            <origin xyz="0.24 0 0" rpy="0 0 0"/>
-        </xacro:inertial_sphere>
-    </link>
-    <xacro:property name="camera_link" value="0.05" /> <!-- Size of square 'camera' box -->
-    <joint name="camera_joint" type="fixed">
-        <axis xyz="0 1 0" />
-        <origin xyz="0.2 0.0 0.1" rpy="0 0 0"/>
-        <parent link="base_link"/>
-        <child link="vanir/base_link/depth_camera1"/>
-    </joint>
-    <!-- Camera -->
-    <link name="vanir/base_link/depth_camera1">
-        <collision>
-        <origin xyz="0 0 0" rpy="0 0 0"/>
-        <geometry>
-        <box size="${camera_link} ${camera_link} ${camera_link}"/>
-        </geometry>
-        </collision>
-        <visual>
-        <origin xyz="0 0 0" rpy="0 0 0"/>
-        <geometry>
-        <box size="${camera_link} ${camera_link} ${camera_link}"/>
-        </geometry>
-        <material name="red"/>
-        </visual>
-        <inertial>
-        <mass value="1e-5" />
-        <origin xyz="0 0 0" rpy="0 0 0"/>
-        <inertia ixx="1e-6" ixy="0" ixz="0" iyy="1e-6" iyz="0" izz="1e-6" />
-        </inertial>
-    </link>
- <!-- LIDAR SENSOR -->
-    <joint name="lidar_joint" type="fixed">
-        <parent link="base_link"/>
-        <child link="vanir/base_link/gpu_lidar"/>
-        <origin xyz="0.04 0 0.18" rpy="0 0 0"/>
-    </joint>
-    <link name="vanir/base_link/gpu_lidar">
-        <visual>
-            <geometry>
-                <cylinder radius="0.03" length="0.06"/>
-            </geometry>
-            <material name="black"/>
-        </visual>
-        <collision>
-            <geometry>
-                <cylinder radius="0.03" length="0.06"/>
-            </geometry>
-        </collision>
-        <inertial>
-            <mass value="0.05"/>
-            <origin xyz="0 0 0" rpy="0 0 0"/>
-            <inertia ixx="1e-6" ixy="0" ixz="0" iyy="1e-6" iyz="0" izz="1e-6"/>
-        </inertial>
-    </link>
+</link>
+  <joint name="camera_joint" type="fixed">
+    <origin xyz="0.000218796 -0.00755 0.0" rpy="0 0 0"/>
+    <parent link="base_link"/>
+    <child link="vanir/base_link/depth_camera1"/>
+  </joint>
+  <!-- LIDAR LINK -->
+  <link name="vanir/base_link/gpu_lidar">
+    <visual>
+      <origin xyz="0.000218796 4.86233e-05 0.000920176" rpy="0 0 0"/>
+      <geometry>
+        <mesh filename="file://$(find vanir_description)/meshes/lidar.stl"/>
+      </geometry>
+      <material name="lidar_material">
+        <color rgba="0.231373 0.380392 0.705882 1.0"/>
+      </material>
+    </visual>
+    <collision>
+      <origin xyz="0.000218796 4.86233e-05 0.000920176" rpy="0 0 0"/>
+      <geometry>
+        <mesh filename="file://$(find vanir_description)/meshes/lidar.stl"/>
+      </geometry>
+    </collision>
+  </link>
+  <joint name="lidar_joint" type="fixed">
+    <origin xyz="0.000218796 4.86233e-05 0.000920176" rpy="0 0 0"/>
+    <parent link="base_link"/>
+    <child link="vanir/base_link/gpu_lidar"/>
+  </joint>
 </robot>
