Commit message: fixed urdf orientation but odom is still flipped

File: vanir_description/urdf/gazebo_control.xacro (robot description, xacro)
@@ -29,6 +29,6 @@
 			<left_joint>wheel_l</left_joint>
     		<right_joint>wheel_r</right_joint>
-    		<wheel_separation>0.45</wheel_separation>
-    		<wheel_radius>0.06</wheel_radius>
+    		<wheel_separation>0.325</wheel_separation>
+    		<wheel_radius>0.145</wheel_radius>
 			<topic>cmd_vel</topic>
     	</plugin>
@@ -48,4 +48,5 @@
 <plugin filename="gz-harmonic-camera-system" name="gz::harmonic::systems::CameraSystem"/>
     <sensor type="camera" name="camera">
+     <pose relative_to='vanir/base_link/depth_camera1'>0.35 0.00 0.1 0 0 0</pose>
       <visualize>true</visualize>
       <always_on>true</always_on>

File: vanir_description/urdf/robot_core.xacro (robot description, xacro)
@@ -1,45 +1,13 @@
 <?xml version="1.0"?>
-<robot xmlns:xacro="http://www.ros.org/wiki/xacro" >
+<robot xmlns:xacro="http://www.ros.org/wiki/xacro" name="vanir_rotated">
   <link name="base_link">
     <inertial>
-      <origin xyz="0.000219763 -0.000623028 0.0710795" rpy="0 0 0"/>
-      <mass value="92.4179"/>
-      <inertia ixx="3.16969" ixy="2.70317e-05" ixz="1.26673e-06" iyy="1.30381" iyz="0.00479148" izz="3.85167"/>
+      <origin xyz="0.0691514 0.00840293 0.0780423" rpy="0 0 0"/>
+      <mass value="86.4984"/>
+      <inertia ixx="1.23316" ixy="-2.70276e-05" ixz="-0.00435928" iyy="2.75808" iyz="1.88929e-06" izz="3.50466"/>
     </inertial>
-    <!-- Part front_caster -->
-    <visual>
-      <origin xyz="0.000218796 0.00283755 0.000920176" rpy="0 -0 0"/>
-      <geometry>
-        <mesh filename="file://$(find vanir_description)/meshes/front_caster.stl"/>
-      </geometry>
-      <material name="front_caster_material">
-        <color rgba="0.301961 0.301961 0.301961 1.0"/>
-      </material>
-    </visual>
-    <collision>
-      <origin xyz="0.000218796 0.00283755 0.000920176" rpy="0 -0 0"/>
-      <geometry>
-        <mesh filename="file://$(find vanir_description)/meshes/front_caster.stl"/>
-      </geometry>
-    </collision>
-    <!-- Part rear_caster -->
-    <visual>
-      <origin xyz="0.000218796 0.00276511 0.000920176" rpy="0 -0 0"/>
-      <geometry>
-        <mesh filename="file://$(find vanir_description)/meshes/rear_caster.stl"/>
-      </geometry>
-      <material name="rear_caster_material">
-        <color rgba="0.301961 0.301961 0.301961 1.0"/>
-      </material>
-    </visual>
-    <collision>
-      <origin xyz="0.000218796 0.00276511 0.000920176" rpy="0 -0 0"/>
-      <geometry>
-        <mesh filename="file://$(find vanir_description)/meshes/rear_caster.stl"/>
-      </geometry>
-    </collision>
     <!-- Part base_link -->
     <visual>
-      <origin xyz="0.000218796 4.86233e-05 0.000920176" rpy="0 -0 0"/>
+      <origin xyz="0.0684338 0.00840189 0.000920176" rpy="0 -0 1.5708"/>
       <geometry>
         <mesh filename="file://$(find vanir_description)/meshes/base_link.stl"/>
@@ -50,5 +18,5 @@
     </visual>
     <collision>
-      <origin xyz="0.000218796 4.86233e-05 0.000920176" rpy="0 -0 0"/>
+      <origin xyz="0.0684338 0.00840189 0.000920176" rpy="0 -0 1.5708"/>
       <geometry>
         <mesh filename="file://$(find vanir_description)/meshes/base_link.stl"/>
@@ -56,13 +24,13 @@
     </collision>
   </link>
-  <!-- Link dof_wheel_r -->
+  <!-- Right Wheel -->
   <link name="dof_wheel_r">
     <inertial>
-      <origin xyz="3.28288e-18 -8.8737e-19 -0.025" rpy="0 0 0"/>
+      <origin xyz="-1.05949e-17 -8.8737e-19 -0.025" rpy="0 0 0"/>
       <mass value="0.908215"/>
-      <inertia ixx="0.00138266" ixy="0" ixz="0" iyy="0.00138266" iyz="0" izz="0.0023869"/>
+      <inertia ixx="0.00138266" ixy="0" ixz="5.88417e-35" iyy="0.00138266" iyz="0" izz="0.0023869"/>
     </inertial>
     <visual>
-      <origin xyz="0 -4.44523e-18 0.1625" rpy="-1.5708 -1.5708 0"/>
+      <origin xyz="-1.38778e-17 -4.44523e-18 0.1625" rpy="-1.5708 -1.5708 0"/>
       <geometry>
         <mesh filename="file://$(find vanir_description)/meshes/dof_wheel_r.stl"/>
@@ -73,5 +41,5 @@
     </visual>
     <collision>
-      <origin xyz="0 -4.44523e-18 0.1625" rpy="-1.5708 -1.5708 0"/>
+      <origin xyz="-1.38778e-17 -4.44523e-18 0.1625" rpy="-1.5708 -1.5708 0"/>
       <geometry>
         <mesh filename="file://$(find vanir_description)/meshes/dof_wheel_r.stl"/>
@@ -80,16 +48,16 @@
   </link>
   <joint name="wheel_r" type="continuous">
-    <origin xyz="-0.162281 4.86233e-05 -0.005" rpy="1.5708 -0 1.5708"/>
+    <origin xyz="0.0684338 -0.154098 -0.0025" rpy="1.5708 -0 3.14159"/>
     <parent link="base_link"/>
     <child link="dof_wheel_r"/>
-    <axis xyz="0 0 1"/>
+    <axis xyz="0 0 -1"/>
     <limit effort="10" velocity="10"/>
   </joint>
-  <!-- Link dof_wheel_l -->
+  <!-- Left Wheel -->
   <link name="dof_wheel_l">
     <inertial>
       <origin xyz="-3.28288e-18 -1.9388e-18 -0.025" rpy="0 0 0"/>
       <mass value="0.908215"/>
-      <inertia ixx="0.00138266" ixy="0" ixz="0" iyy="0.00138266" iyz="0" izz="0.0023869"/>
+      <inertia ixx="0.00138266" ixy="0" ixz="-5.88417e-35" iyy="0.00138266" iyz="0" izz="0.0023869"/>
     </inertial>
     <visual>
@@ -110,37 +78,37 @@
   </link>
   <joint name="wheel_l" type="continuous">
-    <origin xyz="0.162719 4.86233e-05 -0.005" rpy="-1.5708 -0 1.5708"/>
+    <origin xyz="0.0684338 0.170902 -0.0025" rpy="-1.5708 -0 3.14159"/>
     <parent link="base_link"/>
     <child link="dof_wheel_l"/>
-    <axis xyz="0 0 -1"/>
+    <axis xyz="0 0 1"/>
     <limit effort="10" velocity="10"/>
   </joint>
-  <!-- CAMERA LINK -->
-<link name="vanir/base_link/depth_camera1">
-  <visual>
-    <origin xyz="0 0 0" rpy="0 0 0"/>
-    <geometry>
-      <mesh filename="file://$(find vanir_description)/meshes/camera.stl"/>
-    </geometry>
-    <material name="camera_material">
-      <color rgba="0.301961 0.290196 0.262745 1.0"/>
-    </material>
-  </visual>
-  <collision>
-    <origin xyz="0 0 0" rpy="0 0 0"/>
-    <geometry>
-      <mesh filename="file://$(find vanir_description)/meshes/camera.stl"/>
-    </geometry>
-  </collision>
-</link>
+  <!-- Camera -->
+  <link name="vanir/base_link/depth_camera1">
+    <visual>
+      <origin xyz="0.0760324 0.00840189 0.000920176" rpy="0 0 1.5708"/>
+      <geometry>
+        <mesh filename="file://$(find vanir_description)/meshes/camera.stl"/>
+      </geometry>
+      <material name="camera_material">
+        <color rgba="0.301961 0.290196 0.262745 1.0"/>
+      </material>
+    </visual>
+    <collision>
+      <origin xyz="0.0760324 0.00840189 0.000920176" rpy="0 0 1.5708"/>
+      <geometry>
+        <mesh filename="file://$(find vanir_description)/meshes/camera.stl"/>
+      </geometry>
+    </collision>
+  </link>
   <joint name="camera_joint" type="fixed">
-    <origin xyz="0.000218796 -0.00755 0.0" rpy="0 0 0"/>
     <parent link="base_link"/>
     <child link="vanir/base_link/depth_camera1"/>
+    <origin xyz="0.008 0.0 0.001" rpy="0 0 0"/>
   </joint>
-  <!-- LIDAR LINK -->
+  <!-- Lidar -->
   <link name="vanir/base_link/gpu_lidar">
     <visual>
-      <origin xyz="0.000218796 4.86233e-05 0.000920176" rpy="0 0 0"/>
+      <origin xyz="0.0684338 0.00840189 0.000920176" rpy="0 0 1.5708"/>
       <geometry>
         <mesh filename="file://$(find vanir_description)/meshes/lidar.stl"/>
@@ -151,5 +119,5 @@
     </visual>
     <collision>
-      <origin xyz="0.000218796 4.86233e-05 0.000920176" rpy="0 0 0"/>
+      <origin xyz="0.0684338 0.00840189 0.000920176" rpy="0 0 1.5708"/>
       <geometry>
         <mesh filename="file://$(find vanir_description)/meshes/lidar.stl"/>
@@ -158,7 +126,69 @@
   </link>
   <joint name="lidar_joint" type="fixed">
-    <origin xyz="0.000218796 4.86233e-05 0.000920176" rpy="0 0 0"/>
     <parent link="base_link"/>
     <child link="vanir/base_link/gpu_lidar"/>
+    <origin xyz="-0.008 0.0 0.000920176" rpy="0 0 0"/>
   </joint>
+  <!-- Front Caster Link -->
+<link name="front_caster">
+  <visual>
+    <origin xyz="0 0 0" rpy="0 0 0"/>
+    <geometry>
+      <mesh filename="file://$(find vanir_description)/meshes/front_caster.stl"/>
+    </geometry>
+    <material name="front_caster_material">
+      <color rgba="0.301961 0.301961 0.301961 1.0"/>
+    </material>
+  </visual>
+  <collision>
+    <origin xyz="0 0 0" rpy="0 0 0"/>
+    <geometry>
+      <mesh filename="file://$(find vanir_description)/meshes/front_caster.stl"/>
+    </geometry>
+  </collision>
+</link>
+<!-- Joint connecting front caster to base_link -->
+<joint name="front_caster_joint" type="fixed">
+  <origin xyz="0.0656448 0.00840189 0.000920176" rpy="0 -0 1.5708"/>
+  <parent link="base_link"/>
+  <child link="front_caster"/>
+</joint>
+<!-- Rear Caster Link -->
+<link name="rear_caster">
+  <visual>
+    <origin xyz="0 0 0" rpy="0 0 0"/>
+    <geometry>
+      <mesh filename="file://$(find vanir_description)/meshes/rear_caster.stl"/>
+    </geometry>
+    <material name="rear_caster_material">
+      <color rgba="0.301961 0.301961 0.301961 1.0"/>
+    </material>
+  </visual>
+  <collision>
+    <origin xyz="0 0 0" rpy="0 0 0"/>
+    <geometry>
+      <mesh filename="file://$(find vanir_description)/meshes/rear_caster.stl"/>
+    </geometry>
+  </collision>
+</link>
+<!-- Joint connecting rear caster to base_link -->
+<joint name="rear_caster_joint" type="fixed">
+  <origin xyz="0.0657173 0.00840189 0.000920176" rpy="0 -0 1.5708"/>
+  <parent link="base_link"/>
+  <child link="rear_caster"/>
+</joint>
+<gazebo reference="rear_caster">
+  <mu1>2.0</mu1>
+  <mu2>2.0</mu2>
+  <kp>100000.0</kp>
+  <kd>1.0</kd>
+  <material>Gazebo/Black</material>
+</gazebo>
+<gazebo reference="front_caster">
+  <mu1>2.0</mu1>
+  <mu2>2.0</mu2>
+  <kp>100000.0</kp>
+  <kd>1.0</kd>
+  <material>Gazebo/Black</material>
+</gazebo>
 </robot>

Commit message: fixed lidar position

File: vanir_description/urdf/gazebo_control.xacro (robot description, xacro)
@@ -93,5 +93,5 @@
 <gazebo reference="vanir/base_link/gpu_lidar">
   <sensor name='gpu_lidar' type='gpu_lidar'>"
-    <pose relative_to='vanir/base_link/gpu_lidar'>0.001 0.006 0.1155 0 0 0</pose>
+    <pose relative_to='vanir/base_link/gpu_lidar'>0.001 0.006 0.2 0 0 0</pose>
     <frame_id>vanir/base_link/gpu_lidar</frame_id>
     <topic>/laser/scan</topic>

File: vanir_description/urdf/robot_core.xacro (robot description, xacro)
@@ -1,4 +1,4 @@
 <?xml version="1.0"?>
-<robot xmlns:xacro="http://www.ros.org/wiki/xacro" name="vanir_rotated">
+<robot xmlns:xacro="http://www.ros.org/wiki/xacro" name="vanir">
   <link name="base_link">
     <inertial>
@@ -48,5 +48,5 @@
   </link>
   <joint name="wheel_r" type="continuous">
-    <origin xyz="0.0684338 -0.154098 -0.0025" rpy="1.5708 -0 3.14159"/>
+    <origin xyz="0.0684338 -0.2 -0.0025" rpy="1.5708 0 0"/>
     <parent link="base_link"/>
     <child link="dof_wheel_r"/>
@@ -78,5 +78,5 @@
   </link>
   <joint name="wheel_l" type="continuous">
-    <origin xyz="0.0684338 0.170902 -0.0025" rpy="-1.5708 -0 3.14159"/>
+    <origin xyz="0.0684338 0.22 -0.0025" rpy="-1.5708 0 0"/>
     <parent link="base_link"/>
     <child link="dof_wheel_l"/>

Commit message: nav working properly, fixed camera positon

File: vanir_description/urdf/gazebo_control.xacro (robot description, xacro)
@@ -29,5 +29,5 @@
 			<left_joint>wheel_l</left_joint>
     		<right_joint>wheel_r</right_joint>
-    		<wheel_separation>0.325</wheel_separation>
+    		<wheel_separation>0.42</wheel_separation>
     		<wheel_radius>0.145</wheel_radius>
 			<topic>cmd_vel</topic>
@@ -72,4 +72,5 @@
 <gazebo reference="vanir/base_link/depth_camera1">
   <sensor name="depth_camera1" type="depth_camera">
+  <pose relative_to='vanir/base_link/depth_camera1'>0.0 0.3 0.3 0 0 0</pose>
         <always_on>1</always_on>
         <enable_metrics>1</enable_metrics>

File: vanir_description/urdf/robot_core.xacro (robot description, xacro)
@@ -48,5 +48,5 @@
   </link>
   <joint name="wheel_r" type="continuous">
-    <origin xyz="0.0684338 -0.2 -0.0025" rpy="1.5708 0 0"/>
+    <origin xyz="0.0684338 -0.2 -0.0" rpy="1.5708 0 0"/>
     <parent link="base_link"/>
     <child link="dof_wheel_r"/>
@@ -78,5 +78,5 @@
   </link>
   <joint name="wheel_l" type="continuous">
-    <origin xyz="0.0684338 0.22 -0.0025" rpy="-1.5708 0 0"/>
+    <origin xyz="0.0684338 0.22 -0.0" rpy="-1.5708 0 0"/>
     <parent link="base_link"/>
     <child link="dof_wheel_l"/>
@@ -130,13 +130,18 @@
     <origin xyz="-0.008 0.0 0.000920176" rpy="0 0 0"/>
   </joint>
-  <!-- Front Caster Link -->
+<!-- Front Caster Sphere -->
 <link name="front_caster">
+  <inertial>
+    <origin xyz="0 0 0" rpy="0 0 0"/>
+    <mass value="0.1"/>
+    <inertia ixx="1e-5" ixy="0" ixz="0" iyy="1e-5" iyz="0" izz="1e-5"/>
+  </inertial>
   <visual>
     <origin xyz="0 0 0" rpy="0 0 0"/>
     <geometry>
-      <mesh filename="file://$(find vanir_description)/meshes/front_caster.stl"/>
+      <sphere radius="0.07"/>
     </geometry>
-    <material name="front_caster_material">
-      <color rgba="0.301961 0.301961 0.301961 1.0"/>
+    <material name="gray">
+      <color rgba="0.5 0.5 0.5 1.0"/>
     </material>
   </visual>
@@ -144,23 +149,32 @@
     <origin xyz="0 0 0" rpy="0 0 0"/>
     <geometry>
-      <mesh filename="file://$(find vanir_description)/meshes/front_caster.stl"/>
+      <sphere radius="0.07"/>
     </geometry>
   </collision>
 </link>
-<!-- Joint connecting front caster to base_link -->
 <joint name="front_caster_joint" type="fixed">
-  <origin xyz="0.0656448 0.00840189 0.000920176" rpy="0 -0 1.5708"/>
   <parent link="base_link"/>
   <child link="front_caster"/>
+  <origin xyz="0.28 0 0" rpy="0 0 0"/>
 </joint>
-<!-- Rear Caster Link -->
+<gazebo reference="front_caster">
+  <mu1>0.0</mu1>
+  <mu2>0.0</mu2>
+  <material>Gazebo/Gray</material>
+</gazebo>
+<!-- Rear Caster Sphere -->
 <link name="rear_caster">
+  <inertial>
+    <origin xyz="0 0 0" rpy="0 0 0"/>
+    <mass value="0.1"/>
+    <inertia ixx="1e-5" ixy="0" ixz="0" iyy="1e-5" iyz="0" izz="1e-5"/>
+  </inertial>
   <visual>
     <origin xyz="0 0 0" rpy="0 0 0"/>
     <geometry>
-      <mesh filename="file://$(find vanir_description)/meshes/rear_caster.stl"/>
+      <sphere radius="0.07"/>
     </geometry>
-    <material name="rear_caster_material">
-      <color rgba="0.301961 0.301961 0.301961 1.0"/>
+    <material name="gray">
+      <color rgba="0.5 0.5 0.5 1.0"/>
     </material>
   </visual>
@@ -168,27 +182,17 @@
     <origin xyz="0 0 0" rpy="0 0 0"/>
     <geometry>
-      <mesh filename="file://$(find vanir_description)/meshes/rear_caster.stl"/>
+      <sphere radius="0.07"/>
     </geometry>
   </collision>
 </link>
-<!-- Joint connecting rear caster to base_link -->
 <joint name="rear_caster_joint" type="fixed">
-  <origin xyz="0.0657173 0.00840189 0.000920176" rpy="0 -0 1.5708"/>
   <parent link="base_link"/>
   <child link="rear_caster"/>
+  <origin xyz="-0.16 0 0" rpy="0 0 0"/>
 </joint>
 <gazebo reference="rear_caster">
-  <mu1>2.0</mu1>
-  <mu2>2.0</mu2>
-  <kp>100000.0</kp>
-  <kd>1.0</kd>
-  <material>Gazebo/Black</material>
-</gazebo>
-<gazebo reference="front_caster">
-  <mu1>2.0</mu1>
-  <mu2>2.0</mu2>
-  <kp>100000.0</kp>
-  <kd>1.0</kd>
-  <material>Gazebo/Black</material>
+  <mu1>0.0</mu1>
+  <mu2>0.0</mu2>
+  <material>Gazebo/Gray</material>
 </gazebo>
 </robot>

Commit message: fixed odom

File: vanir_description/urdf/gazebo_control.xacro (robot description, xacro)
@@ -27,8 +27,8 @@
 		<plugin filename="gz-sim-diff-drive-system"
 			name="gz::sim::systems::DiffDrive">
-			<left_joint>wheel_l</left_joint>
-    		<right_joint>wheel_r</right_joint>
+			<left_joint>wheel_r</left_joint>
+    		<right_joint>wheel_l</right_joint>
     		<wheel_separation>0.42</wheel_separation>
-    		<wheel_radius>0.145</wheel_radius>
+    		<wheel_radius>0.0725</wheel_radius>
 			<topic>cmd_vel</topic>
     	</plugin>

File: vanir_description/urdf/robot_core.xacro (robot description, xacro)
@@ -47,5 +47,5 @@
     </collision>
   </link>
-  <joint name="wheel_r" type="continuous">
+  <joint name="wheel_l" type="continuous">
     <origin xyz="0.0684338 -0.2 -0.0" rpy="1.5708 0 0"/>
     <parent link="base_link"/>
@@ -77,5 +77,5 @@
     </collision>
   </link>
-  <joint name="wheel_l" type="continuous">
+  <joint name="wheel_r" type="continuous">
     <origin xyz="0.0684338 0.22 -0.0" rpy="-1.5708 0 0"/>
     <parent link="base_link"/>
